Commit message: plugins and rviz in launch files

File: catkin_ws/src/my_robot/urdf/my_robot.xacro (robot description, xacro)
@@ -1,4 +1,5 @@
 <?xml version='1.0'?>
 <robot name="my_robot" xmlns:xacro="http://www.ros.org/wiki/xacro">
+  <xacro:include filename="$(find my_robot)/urdf/my_robot.gazebo" />
   <link name="robot_footprint"></link>
   <joint name="robot_footprint_joint" type="fixed">
@@ -149,5 +150,5 @@
     <axis xyz="0 1 0" rpy="0 0 0"/>
   </joint>
-  <link name='lidar'>
+  <link name='hokuyo'>
     <pose>0 0 0 0 0 0</pose>
     <inertial>
@@ -173,7 +174,7 @@
     </visual>
   </link>
-  <joint type="fixed" name="lidar_joint">
+  <joint type="fixed" name="hokuyo_joint">
     <origin xyz="0.15 0 0.1" rpy="0 0 0"/>
-    <child link="lidar"/>
+    <child link="hokuyo"/>
     <parent link="chassis"/>
     <axis xyz="0 1 0" rpy="0 0 0"/>

Commit message: correction on the robot urdf file and the service is also written

File: catkin_ws/src/my_robot/urdf/my_robot.xacro (robot description, xacro)
@@ -60,5 +60,5 @@
     <inertial>
       <mass value="5.0"/>
-      <origin xyz="0.0 0 0" rpy=" 0 0 0"/>
+      <origin xyz="0.0 0 0" rpy=" 0 1.5707 1.5707"/>
       <inertia
           ixx="0.1" ixy="0" ixz="0"
@@ -68,5 +68,5 @@
     </inertial>
     <collision name='left_wheel_collision'>
-      <origin xyz="0 0 0" rpy=" 0 0 0"/>
+      <origin xyz="0 0 0" rpy=" 0 1.5707 1.5707"/>
       <geometry>
         <cylinder radius="0.1" length="0.05"/>
@@ -74,5 +74,5 @@
     </collision>
     <visual name='left_wheel_visual'>
-      <origin xyz="0 0 0" rpy=" 0 0 0"/>
+      <origin xyz="0 0 0" rpy=" 0 1.5707 1.5707"/>
       <geometry>
         <cylinder radius="0.1" length="0.05"/>
@@ -84,5 +84,5 @@
     <inertial>
       <mass value="5.0"/>
-      <origin xyz="0.0 0 0" rpy=" 0 0 0"/>
+      <origin xyz="0 0 0" rpy=" 0 1.5707 1.5707"/>
       <inertia
           ixx="0.1" ixy="0" ixz="0"
@@ -92,5 +92,5 @@
     </inertial>
     <collision name='right_wheel_collision'>
-      <origin xyz="0 0 0" rpy=" 0 0 0"/>
+      <origin xyz="0 0 0" rpy=" 0 1.5707 1.5707"/>
       <geometry>
         <cylinder radius="0.1" length="0.05"/>
@@ -98,5 +98,5 @@
     </collision>
     <visual name='right_wheel_visual'>
-      <origin xyz="0 0 0" rpy=" 0 0 0"/>
+      <origin xyz="0 0 0" rpy=" 0 1.5707 1.5707"/>
       <geometry>
         <cylinder radius="0.1" length="0.05"/>
@@ -105,5 +105,5 @@
   </link>
   <joint type="continuous" name="left_wheel_hinge">
-    <origin xyz="0 0.15 0" rpy="0 1.5707 1.5707"/>
+    <origin xyz="0 0.15 0" rpy="0 0 0"/>
     <child link="left_wheel"/>
     <parent link="chassis"/>
@@ -113,5 +113,5 @@
   </joint>
   <joint type="continuous" name="right_wheel_hinge">
-    <origin xyz="0 -0.15 0" rpy="0 1.5707 1.5707"/>
+    <origin xyz="0 -0.15 0" rpy="0 0 0"/>
     <child link="right_wheel"/>
     <parent link="chassis"/>

Commit message: colorize my robot

File: catkin_ws/src/my_robot/urdf/my_robot.xacro (robot description, xacro)
@@ -56,4 +56,7 @@
     </visual>
   </link>
+  <gazebo reference="chassis">
+    <material>Gazebo/Blue</material>
+  </gazebo>
   <link name='left_wheel'>
     <pose>0 0 0 0 0 0</pose>
@@ -80,4 +83,7 @@
     </visual>
   </link>
+  <gazebo reference="left_wheel">
+    <material>Gazebo/Green</material>
+  </gazebo>
   <link name='right_wheel'>
     <pose>0 0 0 0 0 0</pose>
@@ -104,4 +110,7 @@
     </visual>
   </link>
+  <gazebo reference="right_wheel">
+    <material>Gazebo/Green</material>
+  </gazebo>
   <joint type="continuous" name="left_wheel_hinge">
     <origin xyz="0 0.15 0" rpy="0 0 0"/>
@@ -144,4 +153,7 @@
     </visual>
   </link>
+  <gazebo reference="camera">
+    <material>Gazebo/Red</material>
+  </gazebo>
   <joint type="fixed" name="camera_joint">
     <origin xyz="0.2 0 0" rpy="0 0 0"/>
